Commit message: Main changes
Lines from Test.py are implemented to Main.py.

File: assets_new/bigrock/bigrock.urdf (robot description, URDF)
Before this commit: robot bigrock, 1 links, 0 joints
Links:
- link baseLink: mass None -> 0.0

File: assets_new/bush/bush.urdf (robot description, URDF)
Before this commit: robot bush, 1 links, 0 joints
Links:
- link baseLink: mass None -> 0.0

File: assets_new/mediumrock/mediumrock.urdf (robot description, URDF)
Before this commit: robot mediumrock, 1 links, 0 joints
Links:
- link baseLink: mass None -> 0.0

File: assets_new/oak/oak.urdf (robot description, URDF)
Before this commit: robot oak, 2 links, 1 joints
Links:
- link baseLink: mass None -> 0.0; geometry collision mesh filename=trunk.obj scale=1 1 1; visual mesh filename=trunk.obj scale=1 1 1
- link leafLink: mass None -> 0.0

File: assets_new/pinusbruita/pinusbruita.urdf (robot description, URDF)
Before this commit: robot pinusbruita, 2 links, 1 joints
Links:
- link baseLink: mass None -> 0.0
- link leafLink: mass None -> 0.0

File: assets_new/smallrock/smallrock.urdf (robot description, URDF)
Before this commit: robot smallrock, 1 links, 0 joints
Links:
- link baseLink: mass None -> 0.0

File: assets_new/tree/tree.urdf (robot description, URDF)
Before this commit: robot tree, 1 links, 0 joints
Links:
- link baseLink: mass None -> 0.0
